Commit message: fix controllers.yaml, ur5.urdf.xacro

File: ur_description/urdf/ur5.urdf.xacro (robot description, xacro)
@@ -46,5 +46,5 @@
     <link name="${prefix}base_link" >
       <visual>
-        <origin xyz="0 0 0" rpy="0 0 ${base_correction}"/>
+        <origin xyz="0 0 0" rpy="0 0 0"/>
         <geometry>
           <mesh filename="package://ur_description/meshes/ur5/visual/base.dae" />
@@ -55,5 +55,5 @@
       </visual>
       <collision>
-        <origin xyz="0 0 0" rpy="0 0 ${base_correction}"/>
+        <origin xyz="0 0 0" rpy="0 0 0"/>
         <geometry>
           <mesh filename="package://ur_description/meshes/ur5/collision/base.stl" />
